File: kicad/teensy-based/usb-teensy_LC_41-theMVP/the_mvp/the_mvp_v1.1.kicad_pcb (KiCad board)
At the start: 2 copper layers, 0 parts

Commit message: adds complete new version of the MVP
Parts:
- added B1: monumentary switch Buttons, Button_Switch_THT:SW_PUSH_6mm_H5mm, F.Cu at (159.0, 70.5)
- added B10: monumentary switch Buttons, Button_Switch_THT:SW_PUSH_6mm_H5mm, F.Cu at (203.5, 145.5)
- added B2: monumentary switch Buttons, Button_Switch_THT:SW_PUSH_6mm_H5mm, F.Cu at (159.0, 83.2)
- added B3: monumentary switch Buttons, Button_Switch_THT:SW_PUSH_6mm_H5mm, F.Cu at (159.0, 95.9)
- added B4: monumentary switch Buttons, Button_Switch_THT:SW_PUSH_6mm_H5mm, F.Cu at (173.8, 70.4)
- added B5: monumentary switch Buttons, Button_Switch_THT:SW_PUSH_6mm_H5mm, F.Cu at (173.7, 83.2)
- added B6: monumentary switch Buttons, Button_Switch_THT:SW_PUSH_6mm_H5mm, F.Cu at (173.7, 95.9)
- added B7: monumentary switch Buttons, Button_Switch_THT:SW_PUSH_6mm_H5mm, F.Cu at (188.5, 70.4)
- added B8: monumentary switch Buttons, Button_Switch_THT:SW_PUSH_6mm_H5mm, F.Cu at (188.5, 83.2)
- added B9: monumentary switch Buttons, Button_Switch_THT:SW_PUSH_6mm_H5mm, F.Cu at (188.3, 95.9)
- added C1: optional, Capacitor_THT:CP_Radial_D10.0mm_P3.50mm, B.Cu at (224.8, 75.4)
- added D1: LED, LED_THT:LED_D5.0mm, F.Cu at (224.0, 87.9)
- added G***: LOGO, Schwurbler:back_print, B.Cu at (153.9, 112.0)
- added G***: LOGO, Schwurbler:frontni, F.Cu at (153.2, 111.8)
- added MCU1: Teensy4.1, Schwurbler:Teensy_Schwurbler_Unified_Footprint, F.Cu at (218.4, 94.9)
- added MHBC: MountingHole_4.3mm_M4, MountingHole:MountingHole_4.3mm_M4, F.Cu at (150.4, 154.9)
- added MHBL: MountingHole_4.3mm_M4, MountingHole:MountingHole_4.3mm_M4, F.Cu at (82.0, 154.9)
- added MHBR: MountingHole_4.3mm_M4, MountingHole:MountingHole_4.3mm_M4, F.Cu at (224.3, 154.9)
- added MHMC: MountingHole_4.3mm_M4, MountingHole:MountingHole_4.3mm_M4, F.Cu at (150.4, 111.0)
- added MHML: MountingHole_4.3mm_M4, MountingHole:MountingHole_4.3mm_M4, F.Cu at (82.0, 111.0)
- added MHMR: MountingHole_4.3mm_M4, MountingHole:MountingHole_4.3mm_M4, F.Cu at (224.3, 111.0)
- added MHTC: MountingHole_4.3mm_M4, MountingHole:MountingHole_4.3mm_M4, F.Cu at (150.4, 67.6)
- added MHTL: MountingHole_4.3mm_M4, MountingHole:MountingHole_4.3mm_M4, F.Cu at (81.8, 67.6)
- added MHTR: MountingHole_4.3mm_M4, MountingHole:MountingHole_4.3mm_M4, F.Cu at (224.3, 67.6)
- added OB1: optional monumentary switch Buttons, Button_Switch_THT:SW_PUSH_6mm_H5mm, F.Cu at (87.6, 70.6)
- added OB2: monumentary switch Button, Button_Switch_THT:SW_PUSH_6mm_H5mm, F.Cu at (87.5, 94.5)
- added OB3: monumentary switch Button, Button_Switch_THT:SW_PUSH_6mm_H5mm, F.Cu at (87.5, 119.5)
- added OB4: monumentary switch Button, Button_Switch_THT:SW_PUSH_6mm_H5mm, F.Cu at (87.5, 144.0)
- added R1: 10kOhm (optional), Resistor_THT:R_Axial_DIN0204_L3.6mm_D1.6mm_P1.90mm_Vertical, B.Cu at (94.2, 80.4)
- added R10: 10kOhm (optional), Resistor_THT:R_Axial_DIN0204_L3.6mm_D1.6mm_P1.90mm_Vertical, B.Cu at (171.1, 98.6)
- added R11: 10kOhm (optional), Resistor_THT:R_Axial_DIN0204_L3.6mm_D1.6mm_P1.90mm_Vertical, B.Cu at (185.9, 73.4)
- added R12: 10kOhm (optional), Resistor_THT:R_Axial_DIN0204_L3.6mm_D1.6mm_P1.90mm_Vertical, B.Cu at (185.4, 88.9)
- added R13: 10kOhm (optional), Resistor_THT:R_Axial_DIN0204_L3.6mm_D1.6mm_P1.90mm_Vertical, B.Cu at (185.7, 99.1)
- added R14: 10kOhm (optional), Resistor_THT:R_Axial_DIN0204_L3.6mm_D1.6mm_P1.90mm_Vertical, B.Cu at (200.5, 148.3)
- added R15: 470Ohm (optional), Resistor_THT:R_Axial_DIN0204_L3.6mm_D1.6mm_P1.90mm_Vertical, B.Cu at (227.1, 92.7)
- added R2: 10kOhm (optional), Resistor_THT:R_Axial_DIN0204_L3.6mm_D1.6mm_P1.90mm_Vertical, B.Cu at (97.5, 98.8)
- added R3: 10kOhm (optional), Resistor_THT:R_Axial_DIN0204_L3.6mm_D1.6mm_P1.90mm_Vertical, B.Cu at (94.1, 129.9)
- added R4: 10kOhm (optional), Resistor_THT:R_Axial_DIN0204_L3.6mm_D1.6mm_P1.90mm_Vertical, B.Cu at (94.4, 154.2)
- added R5: 10kOhm (optional), Resistor_THT:R_Axial_DIN0204_L3.6mm_D1.6mm_P1.90mm_Vertical, B.Cu at (155.8, 73.5)
- added R7: 10kOhm (optional), Resistor_THT:R_Axial_DIN0204_L3.6mm_D1.6mm_P1.90mm_Vertical, B.Cu at (156.0, 98.7)
- added R8: 10kOhm (optional), Resistor_THT:R_Axial_DIN0204_L3.6mm_D1.6mm_P1.90mm_Vertical, B.Cu at (170.3, 73.7)
- added R9: 10kOhm (optional), Resistor_THT:R_Axial_DIN0204_L3.6mm_D1.6mm_P1.90mm_Vertical, B.Cu at (170.3, 88.8)
- added RE1: 10k, Potentiometer_THT:Potentiometer_Alps_RK09K_Single_Vertical, F.Cu at (113.0, 80.0)
- added RE2: 10k, Potentiometer_THT:Potentiometer_Alps_RK09K_Single_Vertical, F.Cu at (113.0, 104.5)
- added RE3: 10k, Potentiometer_THT:Potentiometer_Alps_RK09K_Single_Vertical, F.Cu at (113.0, 129.0)
- added RE4: 10k, Potentiometer_THT:Potentiometer_Alps_RK09K_Single_Vertical, F.Cu at (113.0, 153.7)
- added RE5: 10k, Potentiometer_THT:Potentiometer_Alps_RK09K_Single_Vertical, F.Cu at (137.9, 80.0)
- added RE6: 10k, Potentiometer_THT:Potentiometer_Alps_RK09K_Single_Vertical, F.Cu at (137.3, 104.5)
- added RE7: 10k, Potentiometer_THT:Potentiometer_Alps_RK09K_Single_Vertical, F.Cu at (137.7, 129.0)
- added RE8: 10k, Potentiometer_THT:Potentiometer_Alps_RK09K_Single_Vertical, F.Cu at (138.0, 153.7)
- added RE9: 10k, Potentiometer_THT:Potentiometer_Alps_RK09K_Single_Vertical, F.Cu at (179.3, 139.1)
- added Re: 10kOhm (optional), Resistor_THT:R_Axial_DIN0204_L3.6mm_D1.6mm_P1.90mm_Vertical, B.Cu at (155.8, 85.7)
Routing:
- net Net-(C1-Pad1): track 0.00 -> 548.0 mm, vias 0 -> 1
- net GND: track 0.00 -> 419.0 mm
- net Net-(C1-Pad2): track 0.00 -> 353.7 mm
- net Net-(MCU1-Pad42): track 0.00 -> 162.4 mm
- net Net-(MCU1-Pad5): track 0.00 -> 155.7 mm
- net Net-(MCU1-Pad4): track 0.00 -> 147.7 mm
- net Net-(MCU1-Pad3): track 0.00 -> 134.6 mm
- net Net-(MCU1-Pad44): track 0.00 -> 130.3 mm
- net Net-(MCU1-Pad43): track 0.00 -> 129.6 mm
- net Net-(MCU1-Pad2): track 0.00 -> 124.7 mm
- net Net-(MCU1-Pad38): track 0.00 -> 124.1 mm
- net Net-(MCU1-Pad45): track 0.00 -> 114.1 mm
- net Net-(MCU1-Pad39): track 0.00 -> 99.5 mm
- net Net-(MCU1-Pad41): track 0.00 -> 91.5 mm
- net Net-(MCU1-Pad40): track 0.00 -> 90.8 mm
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- added copper zone on B.Cu, net GND
- added copper zone on F.Cu, net GND
Other:
- board outline added: 153.4 x 98.5 mm
- net class AGND added: clearance 0.2, trace_width 0.5, via_dia 0.8, via_drill 0.4
- net class GND added: clearance 0.2, trace_width 0.5, via_dia 0.8, via_drill 0.4
