File: kicad/MVP/the_mvp_v1.2.kicad_pcb (KiCad board)
At the start: 2 copper layers, 153.4 x 98.5 mm, 52 parts

Commit message: adds code, schematics and pcb
Parts:
- OB1: value optional monumentary switch Buttons -> monumentary switch Button
