File: kicad/Schwurbler-360/schwurbler-360_v1.0_apm_smd.kicad_pcb (KiCad board)
At the start: 2 copper layers, 121.9 x 118.1 mm, 48 parts, among them IC1 MCP23017_SO, SW1 SW_Push, SW2 SW_Push, SW3 SW_Push, SW4 SW_Push, SW5 SW_Push, SW6 SW_Push, SW7 SW_Push, SW8 SW_Push

Commit message: adds schema, pcb and image and cleanup deprecated
Parts:
- added cclogo: LOGO, Schwurbler:ccbyncsa_o, B.Cu at (99.2, 144.2)
- renumbered G*** to 360logo, G*** to smdlogo
