File: kicad/Schwurbler-360/schwurbler-360_v1.0_apm_tth.kicad_pcb (KiCad board)
At the start: 2 copper layers, 121.9 x 118.1 mm, 51 parts, among them IC1 MCP23017_SP, SW1 SW_Push, SW2 SW_Push, SW3 SW_Push, SW4 SW_Push, SW5 SW_Push, SW6 SW_Push, SW7 SW_Push, SW8 SW_Push

Commit message: adds smd edition
Parts:
- added G***: LOGO, Schwurbler:tthedittion, F.Cu at (98.4, 65.1)
- added G***: LOGO, Schwurbler:360, F.Cu at (121.2, 154.3)

Commit message: adds schema, pcb and image and cleanup deprecated
Parts:
- added LOGOcc: LOGO, Schwurbler:ccbyncsa_o, B.Cu at (97.1, 141.3)
- renumbered G*** to logo, G*** to logo360, G*** to logotth
